File: PCB.kicad_sch (KiCad schematic)
At the start: 2 parts

Commit message: trial
Parts:
- removed ?: STM32WBA52CGU6, symbol STM32WBA52CGU6:STM32WBA52CGU6
- added ?: STM32F091RCT6, symbol STM32F091RCT6:STM32F091RCT6
Other:
- moved on the sheet: U?
Changed lines of the file:
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@@
 (kicad_sch (version 20211123) (generator eeschema)
   (paper "A4")
-  (wire (pts (xy 54.61 27.94) (xy 54.61 19.05))
+  (wire (pts (xy 44.45 34.29) (xy 44.45 25.4))
     (stroke (width 0) (type default) (color 0 0 0 0))
   )
-  (wire (pts (xy 97.79 57.15) (xy 92.71 60.96))
+  (wire (pts (xy 181.61 48.26) (xy 185.42 48.26))
     (stroke (width 0) (type default) (color 0 0 0 0))
   )
-  (wire (pts (xy 207.01 71.12) (xy 105.41 72.39))
+  (wire (pts (xy 181.61 50.8) (xy 186.69 50.8))
     (stroke (width 0) (type default) (color 0 0 0 0))
   )
-  (wire (pts (xy 201.93 44.45) (xy 205.74 44.45))
-    (stroke (width 0) (type default) (color 0 0 0 0))
-  )
-  (wire (pts (xy 105.41 72.39) (xy 105.41 59.69))
-    (stroke (width 0) (type default) (color 0 0 0 0))
-  )
-  (wire (pts (xy 97.79 57.15) (xy 143.51 57.15))
-    (stroke (width 0) (type default) (color 0 0 0 0))
-  )
-  (wire (pts (xy 207.01 46.99) (xy 207.01 71.12))
-    (stroke (width 0) (type default) (color 0 0 0 0))
-  )
-  (wire (pts (xy 105.41 59.69) (xy 97.79 59.69))
-    (stroke (width 0) (type default) (color 0 0 0 0))
-  )
-  (wire (pts (xy 34.29 19.05) (xy 54.61 19.05))
-    (stroke (width 0) (type default) (color 0 0 0 0))
-  )
-  (wire (pts (xy 143.51 24.13) (xy 205.74 24.13))
-    (stroke (width 0) (type default) (color 0 0 0 0))
-  )
-  (wire (pts (xy 143.51 57.15) (xy 143.51 24.13))
-    (stroke (width 0) (type default) (color 0 0 0 0))
-  )
-  (wire (pts (xy 97.79 59.69) (xy 92.71 63.5))
-    (stroke (width 0) (type default) (color 0 0 0 0))
-  )
-  (wire (pts (xy 205.74 24.13) (xy 205.74 44.45))
-    (stroke (width 0) (type default) (color 0 0 0 0))
-  )
-  (wire (pts (xy 201.93 46.99) (xy 207.01 46.99))
-    (stroke (width 0) (type default) (color 0 0 0 0))
-  )
-  (symbol (lib_id "power:+5V") (at 34.29 19.05 0) (unit 1)
+  (symbol (lib_id "STM32F091RCT6:STM32F091RCT6") (at 36.83 57.15 0) (unit 1)
     (in_bom yes) (on_board yes) (fields_autoplaced)
-    (property "Reference" "#PWR?" (id 0) (at 34.29 22.86 0)
+    (property "Reference" "?" (id 0) (at 93.98 45.4912 0))
+    (property "Value" "STM32F091RCT6" (id 1) (at 93.98 48.0312 0))
+    (property "Footprint" "" (id 2) (at 36.83 57.15 0)
       (effects (font (size 1.27 1.27)) hide)
     )
-    (property "Value" "+5V" (id 1) (at 34.29 13.97 0))
-    (property "Footprint" "" (id 2) (at 34.29 19.05 0)
+    (property "Datasheet" "" (id 3) (at 36.83 57.15 0)
       (effects (font (size 1.27 1.27)) hide)
     )
-    (property "Datasheet" "" (id 3) (at 34.29 19.05 0)
-      (effects (font (size 1.27 1.27)) hide)
-    )
-    (pin "1")
-  )
-  (symbol (lib_id "STM32WBA52CGU6:STM32WBA52CGU6") (at 46.99 48.26 0) (unit 1)
-    (in_bom yes) (on_board yes)
-    (property "Reference" "?" (id 0) (at 102.87 32.7912 0))
-    (property "Value" "STM32WBA52CGU6" (id 1) (at 102.87 35.3312 0))
-    (property "Footprint" "" (id 2) (at 46.99 48.26 0)
-      (effects (font (size 1.27 1.27)) hide)
-    )
-    (property "Datasheet" "" (id 3) (at 46.99 48.26 0)
-      (effects (font (size 1.27 1.27)) hide)
-    )
-    (property "Reference_1" "IC" (id 4) (at 102.87 37.8712 0))
-    (property "Value_1" "STM32WBA52CGU6" (id 5) (at 102.87 40.4112 0))
-    (property "Footprint_1" "QFN50P700X700X65-49N-D" (id 6) (at 88.9 130.48 0)
+    (property "Reference_1" "IC" (id 4) (at 93.98 50.5712 0))
+    (property "Value_1" "STM32F091RCT6" (id 5) (at 93.98 53.1112 0))
+    (property "Footprint_1" "QFP50P1200X1200X160-64N" (id 6) (at 86.36 136.83 0)
       (effects (font (size 1.27 1.27)) (justify left top) hide)
     )
-    (property "Datasheet_1" "https://www.st.com/resource/en/datasheet/stm32wba52ce.pdf" (id 7) (at 88.9 230.48 0)
+    (property "Datasheet_1" "http://www.st.com/content/ccc/resource/technical/document/datasheet/95/3c/2e/5b/21/09/45/a6/DM00115237.pdf/files/DM00115237.pdf/jcr:content/translations/en.DM00115237.pdf" (id 7) (at 86.36 236.83 0)
       (effects (font (size 1.27 1.27)) (justify left top) hide)
     )
-    (property "Height" "0.65" (id 8) (at 88.9 430.48 0)
+    (property "Height" "1.6" (id 8) (at 86.36 436.83 0)
       (effects (font (size 1.27 1.27)) (justify left top) hide)
     )
-    (property "Manufacturer_Name" "STMicroelectronics" (id 9) (at 88.9 530.48 0)
+    (property "Mouser Part Number" "511-STM32F091RCT6" (id 9) (at 86.36 536.83 0)
       (effects (font (size 1.27 1.27)) (justify left top) hide)
     )
-    (property "Manufacturer_Part_Number" "STM32WBA52CGU6" (id 10) (at 88.9 630.48 0)
+    (property "Mouser Price/Stock" "https://www.mouser.co.uk/ProductDetail/STMicroelectronics/STM32F091RCT6?qs=ClYTdQWm4hDCc82GnPpqOQ%3D%3D" (id 10) (at 86.36 636.83 0)
       (effects (font (size 1.27 1.27)) (justify left top) hide)
     )
-    (property "Mouser Part Number" "511-STM32WBA52CGU6" (id 11) (at 88.9 730.48 0)
+    (property "Manufacturer_Name" "STMicroelectronics" (id 11) (at 86.36 736.83 0)
       (effects (font (size 1.27 1.27)) (justify left top) hide)
     )
-    (property "Mouser Price/Stock" "https://www.mouser.co.uk/ProductDetail/STMicroelectronics/STM32WBA52CGU6?qs=amGC7iS6iy8UV0f66sCfDw%3D%3D" (id 12) (at 88.9 830.48 0)
-      (effects (font (size 1.27 1.27)) (justify left top) hide)
-    )
-    (property "Arrow Part Number" "" (id 13) (at 88.9 930.48 0)
-      (effects (font (size 1.27 1.27)) (justify left top) hide)
-    )
-    (property "Arrow Price/Stock" "" (id 14) (at 88.9 1030.48 0)
+    (property "Manufacturer_Part_Number" "STM32F091RCT6" (id 12) (at 86.36 836.83 0)
       (effects (font (size 1.27 1.27)) (justify left top) hide)
     )
@@
     (pin "49")
     (pin "5")
+    (pin "50")
+    (pin "51")
+    (pin "52")
+    (pin "53")
+    (pin "54")
+    (pin "55")
+    (pin "56")
+    (pin "57")
+    (pin "58")
+    (pin "59")
     (pin "6")
+    (pin "60")
+    (pin "61")
+    (pin "62")
+    (pin "63")
+    (pin "64")
     (pin "7")
     (pin "8")
     (pin "9")
   )
-  (symbol (lib_id "2023-09-13_16-10-09:LSM6DSV16BX") (at 151.13 44.45 0) (unit 1)
+  (symbol (lib_id "2023-09-13_16-10-09:LSM6DSV16BX") (at 130.81 48.26 0) (unit 1)
     (in_bom yes) (on_board yes) (fields_autoplaced)
-    (property "Reference" "U?" (id 0) (at 176.53 33.02 0)
+    (property "Reference" "U?" (id 0) (at 156.21 36.83 0)
       (effects (font (size 1.524 1.524)))
     )
-    (property "Value" "LSM6DSV16BX" (id 1) (at 176.53 36.83 0)
+    (property "Value" "LSM6DSV16BX" (id 1) (at 156.21 40.64 0)
       (effects (font (size 1.524 1.524)))
     )
-    (property "Footprint" "LGA14L_2P59X3P1X0P5_STM" (id 2) (at 151.13 44.45 0)
+    (property "Footprint" "LGA14L_2P59X3P1X0P5_STM" (id 2) (at 130.81 48.26 0)
       (effects (font (size 1.27 1.27) italic) hide)
     )
-    (property "Datasheet" "LSM6DSV16BX" (id 3) (at 151.13 44.45 0)
+    (property "Datasheet" "LSM6DSV16BX" (id 3) (at 130.81 48.26 0)
       (effects (font (size 1.27 1.27) italic) hide)
     )
@@
   )
   (symbol_instances
-    (path "/5a3bcb1e-9cbb-4986-a9af-c07dd118d1d3"
-      (reference "#PWR?") (unit 1) (value "+5V") (footprint "")
-    )
-    (path "/c220eee7-76dd-45ab-b92e-b1db81d2c78d"
-      (reference "?") (unit 1) (value "STM32WBA52CGU6") (footprint "")
+    (path "/b4ef2eba-692d-4b67-aa1b-216fc5f33104"
+      (reference "?") (unit 1) (value "STM32F091RCT6") (footprint "")
     )
     (path "/d806f0ea-4a97-4788-a9ef-11e41d18192a"

Commit message: new stuff
Parts:
- removed U?: LSM6DSV16BX, LGA14L_2P59X3P1X0P5_STM, symbol 2023-09-13_16-10-09:LSM6DSV16BX
- added C1: 10u, symbol Device:C
- added C2, C3, C4, C5: 100n, symbol Device:C
- added U?: RN4871, RF_Module:Microchip_RN4871, symbol RF_Bluetooth:RN4871
- added U?: LSM6DSV16XTR, LGA14L_LSM6_STM, symbol LSM6DSV16XTR:LSM6DSV16XTR
Connections:
- net GND: now reaches ?.12 (VSSA)
- net GND: now also ?.18 (VSS_1), ?.31 (VSS_2), ?.47 (VSS_3), ?.63 (VSS_4), U?.13 (GND), U?.2 (GND), U?.6 (GND), U?.7 (GND)
- net VCC: now reaches ?.19 (VDD_1)
- net VCC: now also ?.32 (VDD_2), ?.64 (VDD_3), C1.1, C2.1, C3.1, C4.1, C5.1, U?.14 (VBAT), U?.8 (VDD)
- net at ?.29 (PB10): now also U?.13 (SCL)
- net at ?.30 (PB11): now also U?.14 (SDA)
- net at ?.42 (PA9): now also U?.8 (UART_TX)
- net at ?.43 (PA10): now also U?.7 (UART_RX)
- new net: C1.2, C2.2, C3.2, C4.2, C5.2
Other:
- moved on the sheet: ?
