File: Battery + Boost/BoostCircuit.kicad_pcb (KiCad board)
At the start: 2 copper layers, 30 x 30 mm, 5 parts, among them U1 TPS610995DRVR

Commit message: Ordered
Parts:
- added J1: Conn_01x04_Pin, Connector_PinHeader_2.54mm:PinHeader_1x04_P2.54mm_Vertical, F.Cu at (122.5, 107.7)
- added J2: Conn_01x04_Pin, Connector_PinHeader_2.54mm:PinHeader_1x04_P2.54mm_Vertical, F.Cu at (144.0, 100.1)
- moved L1 11.4 mm to (135.5, 104.3)
- moved B1 10.9 mm to (132.2, 102.4)
- moved U1 10.9 mm to (132.0, 104.5)
- moved C1 10.9 mm to (133.0, 102.4)
- moved C2 10.9 mm to (129.5, 103.9)
Connections:
- U1 pad V: (no net) -> GND
Routing:
- net GND: track 6.29 -> 27.5 mm, vias 3 -> 2
- net /Vout+: track 3.52 -> 17.0 mm
- net Net-(U1-EN): track 35.4 -> 44.2 mm
- added copper zone on F.Cu, net /Vout+
- added copper zone on F.Cu, net GND
- added copper zone on F.Cu, net Net-(U1-EN)
- added copper zone on F.Cu, net Net-(U1-SW)
- removed copper zone on B.Cu, net GND
Other:
- board text added: "Power PCBv1 ECE 477 Grp 17 Hayagreev, Maham, Patrick, Samantha"
- board text removed: "Power PCB ECE 477 Grp 17 Hayagreev, Maham, Patrick, Samantha"

Commit message: final
Parts:
- C1: footprint Capacitor_SMD:C_0402_1005Metric -> Capacitor_SMD:C_0805_2012Metric
- C2: footprint Capacitor_SMD:C_0402_1005Metric -> Capacitor_SMD:C_1206_3216Metric
- moved C1 1.18 mm to (133.1, 101.2)
- moved J2 0.96 mm to (144.0, 99.2)
- moved C2 0.76 mm to (128.8, 104.0)
- moved J1 0.44 mm to (122.5, 107.3)
Routing:
- net GND: track 27.5 -> 37.9 mm
- net Net-(U1-EN): track 44.2 -> 49.3 mm
