File: Battery + Boost/BoostCircuit.kicad_sch (KiCad schematic)
At the start: 5 parts, among them U1 TPS610995DRVR

Commit message: Ordered
Parts:
- added J1: Conn_01x04_Pin, Connector_PinHeader_2.54mm:PinHeader_1x04_P2.54mm_Vertical, symbol Connector:Conn_01x04_Pin
Connections:
- net GND: now also J1.1 (Pin_1), J1.4 (Pin_4)
- net Vout+: now also J1.2 (Pin_2), J1.3 (Pin_3)
Changed lines of the file:
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@@
   (junction (at 99.06 86.36) (diameter 0) (color 0 0 0 0)
   )
-  (junction (at 66.04 91.44) (diameter 0) (color 0 0 0 0)
-  )
   (junction (at 152.4 86.36) (diameter 0) (color 0 0 0 0)
   )
+  (junction (at 175.26 93.98) (diameter 0) (color 0 0 0 0)
+  )
   (junction (at 142.24 111.76) (diameter 0) (color 0 0 0 0)
   )
   (junction (at 91.44 111.76) (diameter 0) (color 0 0 0 0)
   )
+  (junction (at 172.72 99.06) (diameter 0) (color 0 0 0 0)
+  )
+  (junction (at 68.58 86.36) (diameter 0) (color 0 0 0 0)
+  )
   (junction (at 142.24 99.06) (diameter 0) (color 0 0 0 0)
   )
   (junction (at 152.4 111.76) (diameter 0) (color 0 0 0 0)
   )
-  (wire (pts (xy 66.04 91.44) (xy 66.04 93.98))
-    (stroke (width 0) (type default))
-  )
   (wire (pts (xy 68.58 111.76) (xy 68.58 109.22))
     (stroke (width 0) (type default))
@@
     (stroke (width 0) (type default))
   )
-  (wire (pts (xy 66.04 86.36) (xy 66.04 91.44))
-    (stroke (width 0) (type default))
-  )
   (wire (pts (xy 99.06 86.36) (xy 99.06 81.28))
     (stroke (width 0) (type default))
   )
+  (wire (pts (xy 68.58 86.36) (xy 68.58 93.98))
+    (stroke (width 0) (type default))
+  )
+  (wire (pts (xy 165.1 99.06) (xy 172.72 99.06))
+    (stroke (width 0) (type default))
+  )
   (wire (pts (xy 144.78 81.28) (xy 142.24 81.28))
     (stroke (width 0) (type default))
@@
     (stroke (width 0) (type default))
   )
-  (wire (pts (xy 68.58 93.98) (xy 68.58 91.44))
+  (wire (pts (xy 172.72 91.44) (xy 177.8 91.44))
+    (stroke (width 0) (type default))
+  )
+  (wire (pts (xy 177.8 93.98) (xy 175.26 93.98))
+    (stroke (width 0) (type default))
+  )
+  (wire (pts (xy 165.1 86.36) (xy 165.1 93.98))
     (stroke (width 0) (type default))
   )
@@
     (stroke (width 0) (type default))
   )
+  (wire (pts (xy 165.1 111.76) (xy 165.1 99.06))
+    (stroke (width 0) (type default))
+  )
   (wire (pts (xy 152.4 111.76) (xy 142.24 111.76))
     (stroke (width 0) (type default))
@@
     (stroke (width 0) (type default))
   )
+  (wire (pts (xy 66.04 86.36) (xy 66.04 93.98))
+    (stroke (width 0) (type default))
+  )
   (wire (pts (xy 91.44 114.3) (xy 91.44 111.76))
     (stroke (width 0) (type default))
   )
-  (wire (pts (xy 66.04 86.36) (xy 91.44 86.36))
+  (wire (pts (xy 66.04 86.36) (xy 68.58 86.36))
+    (stroke (width 0) (type default))
+  )
+  (wire (pts (xy 165.1 93.98) (xy 175.26 93.98))
     (stroke (width 0) (type default))
   )
@@
     (stroke (width 0) (type default))
   )
+  (wire (pts (xy 172.72 99.06) (xy 172.72 91.44))
+    (stroke (width 0) (type default))
+  )
+  (wire (pts (xy 177.8 99.06) (xy 172.72 99.06))
+    (stroke (width 0) (type default))
+  )
   (wire (pts (xy 104.14 81.28) (xy 99.06 81.28))
     (stroke (width 0) (type default))
   )
+  (wire (pts (xy 175.26 93.98) (xy 175.26 96.52))
+    (stroke (width 0) (type default))
+  )
   (wire (pts (xy 99.06 81.28) (xy 99.06 63.5))
     (stroke (width 0) (type default))
@@
     (stroke (width 0) (type default))
   )
-  (wire (pts (xy 68.58 91.44) (xy 66.04 91.44))
+  (wire (pts (xy 175.26 96.52) (xy 177.8 96.52))
+    (stroke (width 0) (type default))
+  )
+  (wire (pts (xy 68.58 86.36) (xy 91.44 86.36))
     (stroke (width 0) (type default))
   )
@@
   (label "Vout+" (at 165.1 86.36 0) (fields_autoplaced)
     (effects (font (size 1.27 1.27)) (justify left bottom))
+  )
+  (netclass_flag "" (length 2.54) (shape round) (at 78.74 86.36 0) (fields_autoplaced)
+    (effects (font (size 1.27 1.27)) (justify left bottom))
+    (property "Netclass" "Vin" (at 79.4385 83.82 0)
+      (effects (font (size 1.27 1.27) italic) (justify left))
+    )
+  )
+  (netclass_flag "" (length 2.54) (shape round) (at 144.78 63.5 0) (fields_autoplaced)
+    (effects (font (size 1.27 1.27)) (justify left bottom))
+    (property "Netclass" "Vsw" (at 145.4785 60.96 0)
+      (effects (font (size 1.27 1.27) italic) (justify left))
+    )
   )
   (symbol (lib_id "TFM201610GHM-2R2MTAA:TFM201610GHM-2R2MTAA") (at 111.76 63.5 0) (unit 1)
@@
         )
       )
+    )
+  )
+  (symbol (lib_id "Connector:Conn_01x04_Pin") (at 182.88 96.52 180) (unit 1)
+    (in_bom yes) (on_board yes) (dnp no) (fields_autoplaced)
+    (property "Reference" "J1" (at 184.15 93.98 0)
+      (effects (font (size 1.27 1.27)) (justify right))
+    )
+    (property "Value" "Conn_01x04_Pin" (at 184.15 96.52 0)
+      (effects (font (size 1.27 1.27)) (justify right))
+    )
+    (property "Footprint" "Connector_PinHeader_2.54mm:PinHeader_1x04_P2.54mm_Vertical" (at 182.88 96.52 0)
+      (effects (font (size 1.27 1.27)) hide)
+    )
+    (property "Datasheet" "~" (at 182.88 96.52 0)
+      (effects (font (size 1.27 1.27)) hide)
+    )
+    (pin "1")
+    (pin "2")
+    (pin "3")
+    (pin "4")
+    (instances
+      (project "BoostCircuit"
+        (path "/d9f15cc4-04b7-414f-9766-ef396b42d7fe"
+          (reference "J1") (unit 1)
+        )
+      )

Commit message: final
Parts:
- C1: footprint Capacitor_SMD:C_0402_1005Metric -> Capacitor_SMD:C_0805_2012Metric
- C2: footprint Capacitor_SMD:C_0402_1005Metric -> Capacitor_SMD:C_1206_3216Metric
Changed lines of the file:
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@@
       (effects (font (size 1.27 1.27)) (justify left))
     )
-    (property "Footprint" "Capacitor_SMD:C_0402_1005Metric" (at 92.4052 96.52 0)
+    (property "Footprint" "Capacitor_SMD:C_0805_2012Metric" (at 92.4052 96.52 0)
       (effects (font (size 1.27 1.27)) hide)
     )
@@
       (effects (font (size 1.27 1.27)) (justify left))
     )
-    (property "Footprint" "Capacitor_SMD:C_0402_1005Metric" (at 153.3652 99.06 0)
+    (property "Footprint" "Capacitor_SMD:C_1206_3216Metric" (at 153.3652 99.06 0)
       (effects (font (size 1.27 1.27)) hide)
     )
