File: MCU+IMU/MCU+IMU.kicad_sch (KiCad schematic)
At the start: 21 parts, among them J1 Conn_01x04_Male, SW1 SW_Push, U1 LSM6DSV16XTR, U2 STM32F091RCT6, U3 RN4871, U4 MAX7375AXR405

Commit message: Ordered
Parts:
- removed C12: 100n, Capacitor_SMD:C_0402_1005Metric, symbol Device:C
- removed U4: MAX7375AXR405, Package_TO_SOT_SMD:SOT-323_SC-70, symbol Oscillator:MAX7375AXR405
- added J2: Conn_01x04, 4PinConnector:2MMHBS04VT02HTB, symbol Connector_Generic:Conn_01x04
- C1, C10, C11: footprint Capacitor_SMD:C_0603_1608Metric -> Capacitor_SMD:C_0805_2012Metric
- C11, C2, C3, C5, C6, C7, C8, C9: footprint Capacitor_SMD:C_0402_1005Metric -> Capacitor_SMD:C_0805_2012Metric
Connections:
- net GND: now also J2.1 (Pin_1), J2.4 (Pin_4)
- net USART1_RX: now also U2.9 (PC1), U3.8 (UART_TX); no longer U2.42 (PA9), U3.7 (UART_RX)
- net USART1_TX: now also U2.8 (PC0), U3.7 (UART_RX); no longer U2.43 (PA10), U3.8 (UART_TX)
- net VDD: now also U2.48 (VDDIO2), J2.2 (Pin_2), J2.3 (Pin_3)
- net PB12: now reaches U2.33 (PB12)
- net PB13: now reaches U2.34 (PB13)
- net PB14: now reaches U2.35 (PB14)
- net PB15: now reaches U2.36 (PB15)
- net PA11: now reaches U2.44 (PA11)
- net PA12: now reaches U2.45 (PA12)
- net IMU_INT: no longer names the net of U2.27 (PB1)
- net IMU_INT: no longer U1.9 (INT2)
- net MODE_SEL: no longer names the net of U3.16 (P2_0)
- net MODE_SEL: no longer U2.41 (PA8)
- net SI_OSC: no longer names the net of U2.5 (PF0)
- new net PA10: U2.43 (PA10)
- new net PA8: U2.41 (PA8)
- new net PA9: U2.42 (PA9)
- no-connect marks 13 -> 12
Other:
- note removed: "Silicon Oscillator"

Commit message: final
Parts:
- J1, J2: footprint 4PinConnector:2MMHBS04VT02HTB -> Connector_PinHeader_2.54mm:PinHeader_1x04_P2.54mm_Vertical
Changed lines of the file:
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@@
       (effects (font (size 1.27 1.27)) (justify right))
     )
-    (property "Footprint" "4PinConnector:2MMHBS04VT02HTB" (at 144.78 81.28 0)
+    (property "Footprint" "Connector_PinHeader_2.54mm:PinHeader_1x04_P2.54mm_Vertical" (at 144.78 81.28 0)
       (effects (font (size 1.27 1.27)) hide)
     )
@@
       (effects (font (size 1.27 1.27)) (justify left))
     )
-    (property "Footprint" "4PinConnector:2MMHBS04VT02HTB" (at 236.22 139.7 0)
+    (property "Footprint" "Connector_PinHeader_2.54mm:PinHeader_1x04_P2.54mm_Vertical" (at 236.22 139.7 0)
       (effects (font (size 1.27 1.27)) hide)
     )
